Commit message: added gazebo launch

File: my_robot_description/urdf/simple_robot.urdf (robot description, URDF)
Before this commit: robot simple_robot, 1 links, 0 joints
Links:
- added link world
- link base_link: mass None -> 1.0; geometry collision box size=0.1 0.1 0.1; visual box size=0.1 0.1 0.1
Joints:
- added joint base_world: type fixed, parent world, child base_link, origin xyz=0.0 0.0 0.0 rpy=0.0 0.0 0.0
